File: pcb/pos.kicad_sch (KiCad schematic)
At the start: 8 parts, among them J1 UART Debug

Commit message: pcb: swap keypad pins 4 and 7 between GPIO2 and GPIO10 so every key wakes the terminal
Only GPIO0-5 can wake the ESP32-C3 from deep sleep and column 0 (keys
1 4 7 *) sat on GPIO10. The schematic now routes keypad pin 4 (column 0)
to GPIO2 and pin 7 (row 2) to GPIO10; the PCB still needs "Update PCB
from schematic" and two traces rerouted. Firmware picks the pin map by
BOARD_REV (1 = first run, default; 2 = this revision).

Co-Authored-By: Claude Fable 5.1 <noreply@anthropic.com>
Claude-Session: https://claude.ai/code/session_01VMi2Y1oKPZ3TeeFmLej47y
Connections:
- net at KEYPAD1.4 (Pin_4): now also ESP32.1 (GPIO2/A0/D0); no longer ESP32.11 (GPIO10/D10/MOSI)
- net at KEYPAD1.7 (Pin_7): now also ESP32.11 (GPIO10/D10/MOSI); no longer ESP32.1 (GPIO2/A0/D0)
Changed lines of the file:
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@@
 	(wire
 		(pts
-			(xy 127 120.65) (xy 127 140.97)
+			(xy 134.62 120.65) (xy 134.62 140.97)
 		)
 		(stroke
@@
 	(wire
 		(pts
-			(xy 171.45 120.65) (xy 127 120.65)
+			(xy 171.45 120.65) (xy 134.62 120.65)
 		)
 		(stroke
@@
 	(wire
 		(pts
-			(xy 134.62 115.57) (xy 134.62 140.97)
+			(xy 127 115.57) (xy 127 140.97)
 		)
 		(stroke
@@
 	(wire
 		(pts
-			(xy 115.57 115.57) (xy 134.62 115.57)
-		)
-		(stroke
+			(xy 115.57 115.57) (xy 127 115.57)
+		)
+		(stroke
