File: pcb/pos.kicad_pcb (KiCad board)
At the start: 4 copper layers, 60.9 x 111.1 mm, 9 parts, among them U0TXD U0TXD

Commit message: pcb: adopt the live KiCad project (was ~/pos) and the v1/v2 fab gerber zips
~/pos is now a symlink into the repo so KiCad's recent-projects entries
keep working and every save is versioned. The board file carries the
reference re-annotation (KEYPAD1, LED1) from today's netlist sync; the
keypad pin swap still needs Update PCB from Schematic plus two traces.

Co-Authored-By: Claude Fable 5.1 <noreply@anthropic.com>
Claude-Session: https://claude.ai/code/session_01VMi2Y1oKPZ3TeeFmLej47y
Parts:
- J1: renamed from U0TXD; value U0TXD -> UART Debug
- renumbered KEYPAD to KEYPAD1, LED to LED1
Changed lines of the file:
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@@
 	(net 16 "unconnected-(ESP32-VBUS-Pad14)")
 	(net 17 "Net-(ESP32-GPIO21{slash}D6{slash}TX)")
+	(net 18 "unconnected-(ESP32-VBUS-Pad14)_1")
 	(footprint "LED_THT:LED_D5.0mm"
 		(layer "F.Cu")
@@
 		(descr "LED, diameter 5.0mm, 2 pins, http://cdn-reichelt.de/documents/datenblatt/A500/LL-504BC2E-009.pdf, generated by kicad-footprint-generator")
 		(tags "LED")
-		(property "Reference" "LED"
+		(property "Reference" "LED1"
 			(at 1.275 4 0)
 			(layer "F.SilkS")
@@
 		(layer "F.Cu")
 		(at 142.6 109.82)
-		(property "Reference" "KEYPAD"
+		(property "Reference" "KEYPAD1"
 			(at -3.6 2.5 0)
 			(unlocked yes)
@@
 			(layers "B.Cu" "B.Mask")
 			(roundrect_rratio 0.1)
-			(net 16 "unconnected-(ESP32-VBUS-Pad14)")
+			(net 18 "unconnected-(ESP32-VBUS-Pad14)_1")
 			(pinfunction "VBUS")
 			(pintype "passive+no_connect")
@@
 		(descr "Through hole straight pin header, 1x02, 2.54mm pitch, single row")
 		(tags "Through hole pin header THT 1x02 2.54mm single row")
-		(property "Reference" "U0TXD"
+		(property "Reference" "J1"
 			(at -2.5 -0.275 0)
 			(layer "B.SilkS")
@@
 			)
 		)
-		(property "Value" "U0TXD"
+		(property "Value" "UART Debug"
 			(at 3 0.5 0)
 			(layer "B.Fab")
