File: pcb/pos.kicad_pcb (KiCad board)
At the start: 4 copper layers, 60.9 x 111.1 mm, 9 parts, among them J1 UART Debug

Commit message: pcb: reroute keypad pins 4 and 7 for revision 2
Connections:
- KEYPAD1 pad 4: Net-(ESP32-GPIO10/D10/MOSI) -> Net-(ESP32-GPIO2/A0/D0)
- KEYPAD1 pad 7: Net-(ESP32-GPIO2/A0/D0) -> Net-(ESP32-GPIO10/D10/MOSI)
Routing:
- net Net-(ESP32-GPIO2/A0/D0): track 25.0 -> 41.1 mm
- net Net-(ESP32-GPIO10/D10/MOSI): track 19.6 -> 31.3 mm
Changed lines of the file:
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@@
 			(layers "*.Cu" "*.Mask")
 			(remove_unused_layers no)
-			(net 14 "Net-(ESP32-GPIO10{slash}D10{slash}MOSI)")
+			(net 13 "Net-(ESP32-GPIO2{slash}A0{slash}D0)")
 			(pinfunction "Pin_4")
 			(pintype "passive")
@@
 			(layers "*.Cu" "*.Mask")
 			(remove_unused_layers no)
-			(net 13 "Net-(ESP32-GPIO2{slash}A0{slash}D0)")
+			(net 14 "Net-(ESP32-GPIO10{slash}D10{slash}MOSI)")
 			(pinfunction "Pin_7")
 			(pintype "passive")
@@
 	)
 	(segment
-		(start 147.984 141.444)
-		(end 169.996 141.444)
+		(start 156.260578 129.071501)
+		(end 167.629077 140.44)
 		(width 0.127)
 		(layer "F.Cu")
@@
 	)
 	(segment
-		(start 169.996 141.444)
+		(start 150.448499 129.071501)
+		(end 156.260578 129.071501)
+		(width 0.127)
+		(layer "F.Cu")
+		(net 13)
+	)
+	(segment
+		(start 139.22 140.3)
+		(end 150.448499 129.071501)
+		(width 0.127)
+		(layer "F.Cu")
+		(net 13)
+	)
+	(segment
+		(start 167.629077 140.44)
 		(end 171 140.44)
 		(width 0.127)
@@
 	)
 	(segment
+		(start 157.455 130.626547)
+		(end 156.154953 129.3265)
+		(width 0.127)
+		(layer "F.Cu")
+		(net 14)
+	)
+	(segment
+		(start 156.049625 139.410999)
+		(end 157.455 138.005624)
+		(width 0.127)
+		(layer "F.Cu")
+		(net 14)
+	)
+	(segment
+		(start 151.871547 132.82)
+		(end 155.76 132.82)
+		(width 0.127)
+		(layer "F.Cu")
+		(net 14)
+	)
+	(segment
 		(start 146.84 140.3)
 		(end 147.984 141.444)
 		(width 0.127)
 		(layer "F.Cu")
-		(net 13)
+		(net 14)
 	)
 	(segment
-		(start 146.7 132.82)
-		(end 155.76 132.82)
+		(start 147.984 141.444)
+		(end 152.393861 141.444)
 		(width 0.127)
 		(layer "F.Cu")
@@
 	)
 	(segment
-		(start 139.22 140.3)
-		(end 146.7 132.82)
+		(start 156.154953 129.3265)
+		(end 155.365047 129.3265)
+		(width 0.127)
+		(layer "F.Cu")
+		(net 14)
+	)
+	(segment
+		(start 154.426862 139.410999)
+		(end 156.049625 139.410999)
+		(width 0.127)
+		(layer "F.Cu")
+		(net 14)
+	)
+	(segment
+		(start 155.365047 129.3265)
+		(end 151.871547 132.82)
+		(width 0.127)
+		(layer "F.Cu")
+		(net 14)
+	)
+	(segment
+		(start 157.455 138.005624)
+		(end 157.455 130.626547)
+		(width 0.127)
+		(layer "F.Cu")
+		(net 14)
+	)
+	(segment
+		(start 152.393861 141.444)
+		(end 154.426862 139.410999)
 		(width 0.127)
 		(layer "F.Cu")
